Commit message: fix needle orientation

File: demo_staubli_med_2025/urdf/needle_holder.xacro (robot description, xacro)
@@ -5,5 +5,5 @@
         <link name="needle_holder_link">
             <visual>
-                <origin xyz="0 0 0" rpy="0 0 0"/>
+                <origin xyz="0 0 0" rpy="0 0 ${90*pi/180}"/>
                 <geometry>
                     <mesh filename="package://demo_staubli_med_2025/meshes/visual/needle_holder.dae"/>
@@ -11,5 +11,5 @@
             </visual>
             <collision>
-                <origin xyz="0 0 0" rpy="0 0 0"/>
+                <origin xyz="0 0 0" rpy="0 0 ${90*pi/180}"/>
                 <geometry>
                     <mesh filename="package://demo_staubli_med_2025/meshes/collision/needle_holder.stl"/>
@@ -25,5 +25,5 @@
         <link name="needle_link">
             <visual>
-                <origin xyz="0 0 ${-needle_length/2}" rpy="0 0 0"/>
+                <origin xyz="${-needle_length/2} 0 0" rpy="0 ${90*pi/180} 0"/>
                 <geometry>
                     <cylinder radius="0.0025" length="${needle_length}"/>
@@ -53,5 +53,5 @@
         <joint name="needle_visual_joint" type="fixed">
             <!-- % FT sensor : x="59.36" y="0.83" z="157.165" rx="2.25775e-14" ry="65" rz="90" -->
-            <origin xyz="0 ${-needle_length} 0.136" rpy="${90*pi/180} 0 0"/>
+            <origin xyz="${needle_length} 0 0.136" rpy="0 0 0"/>
             <parent link="needle_holder_link" />
             <child link="needle_link" />
